Commit message: add center of gravity and detection parachute (0 mass both for now)

File: models/vehicles/racecar/racecar.urdf (robot description, URDF)
Before this commit: robot racecar, 21 links, 20 joints
Links:
- added link center_of_gravity_link, mass 0.0; collision box size=0.1 0.1 0.1; visual box size=0.1 0.1 0.1
- added link detection_link, mass 0.0; collision box size=0.01 0.175 0.20; visual box size=0.01 0.175 0.20
Joints:
- added joint center_of_gravity_joint: type fixed, parent chassis, child center_of_gravity_link, origin xyz=0.1 0.0 0.075 rpy=0 0 0, axis 0 0 1
- added joint detection_joint: type fixed, parent center_of_gravity_link, child detection_link, origin xyz=-0.05 0.0 0.0 rpy=0 0 0, axis 0 0 1

Commit message: correct scale to 3 values, instead of 4

File: models/vehicles/racecar/racecar.urdf (robot description, URDF)
Before this commit: robot racecar, 23 links, 22 joints
Links:
- link chassis: geometry collision mesh filename=meshes/chassis_differential.STL scale=1 1 1; visual mesh filename=meshes/chassis_differential.STL scale=1 1 1

Commit message: messing up with urdf, change masses messing up with multipliers to get higher speed

File: models/vehicles/racecar/racecar.urdf (robot description, URDF)
Before this commit: robot racecar, 23 links, 22 joints
Links:
- link center_of_gravity_link: mass 0.0 -> 0.50; geometry collision box size=0.05 0.05 0.05; visual box size=0.05 0.05 0.05
- link chassis: mass 4.0 -> 1.44
- link detection_link: mass 0.0 -> 0.01
Joints:
- joint center_of_gravity_joint: origin xyz=0.1 0.0 0.075 rpy=0 0 0 -> xyz=0.17145 0.0 0.01 rpy=0 0 0
- joint detection_joint: origin xyz=-0.05 0.0 0.0 rpy=0 0 0 -> xyz=-0.05 0.0 0.125 rpy=0 0 0; parent center_of_gravity_link -> chassis
- joint hokuyo_joint: origin xyz=0.265 0.0 0.075 rpy=0 0 0 -> xyz=0.335 0.0 0.075 rpy=0 0 0
- joint left_steering_hinge_joint: origin xyz=0.325 0.1 0 rpy=0 1.5708 0 -> xyz=0.3302 0.1 0 rpy=0 1.5708 0
- joint right_steering_hinge_joint: origin xyz=0.325 -0.1 0 rpy=0 1.5708 0 -> xyz=0.3302 -0.1 0 rpy=0 1.5708 0

Commit message: modify parachute to have also side panels

File: models/vehicles/racecar/racecar.urdf (robot description, URDF)
Before this commit: robot racecar, 23 links, 22 joints
Links:
- added link detection_left_link, mass 0.01; collision box size=0.01 0.175 0.10; visual box size=0.01 0.175 0.10
- added link detection_right_link, mass 0.01; collision box size=0.01 0.175 0.10; visual box size=0.01 0.175 0.10
- link detection_link: geometry collision box size=0.01 0.175 0.10; visual box size=0.01 0.175 0.10
Joints:
- added joint detection_left_joint: type fixed, parent detection_link, child detection_left_link, origin xyz=0.0875 0.0875 0.0 rpy=0 0 1.570796, axis 0 0 1
- added joint detection_right_joint: type fixed, parent detection_link, child detection_right_link, origin xyz=0.0875 -0.0875 0.0 rpy=0 0 1.570796, axis 0 0 1
- joint detection_joint: origin xyz=-0.05 0.0 0.125 rpy=0 0 0 -> xyz=-0.05 0.0 0.075 rpy=0 0 0

Commit message: modify laser position after measurements on real car

File: models/vehicles/racecar/racecar.urdf (robot description, URDF)
Before this commit: robot racecar, 25 links, 24 joints
Joints:
- joint hokuyo_joint: origin xyz=0.335 0.0 0.075 rpy=0 0 0 -> xyz=0.217 0.0 0.088 rpy=0 0 0
